File: Electronics/LCP_PowerControl/ActuatorConnector.sch (KiCad schematic (older format))
At the start: 2 parts

Commit message: Aiming for rev 0.1 complete
Parts:
- J17: renamed from J?; footprint (none) -> Connector_Molex:Molex_Micro-Fit_3.0_43045-0200_2x01_P3.00mm_Horizontal
- J18: renamed from J?; footprint (none) -> Connector_Molex:Molex_Micro-Fit_3.0_43045-0400_2x02_P3.00mm_Horizontal
Changed lines of the file:
@@
 Sheet 10 11
 Title ""
-Date ""
-Rev ""
+Date "2020-06-17"
+Rev "R0.1"
 Comp ""
-Comment1 ""
+Comment1 "Design by: Matt Casari"
 Comment2 ""
 Comment3 ""
@@
 P 7450 3150
 AR Path="/5EE2AB43/5EE8A2E1" Ref="J?"  Part="1"
-AR Path="/5EE7B956/5EE8A2E1" Ref="J?"  Part="1"
-F 0 "J?" H 7530 3142 50  0000 L CNN
+AR Path="/5EE7B956/5EE8A2E1" Ref="J17"  Part="1"
+F 0 "J17" H 7530 3142 50  0000 L CNN
 F 1 "Conn_01x02" H 7530 3051 50  0000 L CNN
-F 2 "" H 7450 3150 50  0001 C CNN
+F 2 "Connector_Molex:Molex_Micro-Fit_3.0_43045-0200_2x01_P3.00mm_Horizontal" H 7450 3150 50  0001 C CNN
 F 3 "~" H 7450 3150 50  0001 C CNN
 	1    7450 3150
@@
 	4850 3250 7250 3250
 $Comp
-L Connector_Generic:Conn_01x04 J?
+L Connector_Generic:Conn_01x04 J18
 U 1 1 5EE8A71A
 P 7450 4050
-F 0 "J?" H 7530 4042 50  0000 L CNN
+F 0 "J18" H 7530 4042 50  0000 L CNN
 F 1 "Conn_01x04" H 7530 3951 50  0000 L CNN
-F 2 "" H 7450 4050 50  0001 C CNN
+F 2 "Connector_Molex:Molex_Micro-Fit_3.0_43045-0400_2x02_P3.00mm_Horizontal" H 7450 4050 50  0001 C CNN
 F 3 "~" H 7450 4050 50  0001 C CNN
 	1    7450 4050

Commit message: BOM Update
Updated MPNs on components to match supplies as well as correcting some resistor values
Parts:
- J17: MPN (none) -> 0430450213
- J18: MPN (none) -> 0430450413
Changed lines of the file:
@@
 F 2 "Connector_Molex:Molex_Micro-Fit_3.0_43045-0200_2x01_P3.00mm_Horizontal" H 7450 3150 50  0001 C CNN
 F 3 "~" H 7450 3150 50  0001 C CNN
+F 4 "0430450213" H 7450 3150 50  0001 C CNN "MPN"
 	1    7450 3150
 	1    0    0    -1
@@
 F 2 "Connector_Molex:Molex_Micro-Fit_3.0_43045-0400_2x02_P3.00mm_Horizontal" H 7450 4050 50  0001 C CNN
 F 3 "~" H 7450 4050 50  0001 C CNN
+F 4 "0430450413" H 7450 4050 50  0001 C CNN "MPN"
 	1    7450 4050
 	1    0    0    -1

Commit message: LCP PowerControl Board Update
Parts:
- J17: footprint Connector_Molex:Molex_Micro-Fit_3.0_43045-0200_2x01_P3.00mm_Horizontal -> Connector_Molex:Molex_Micro-Fit_3.0_43045-0212_2x01_P3.00mm_Vertical
Changed lines of the file:
@@
 F 0 "J17" H 7530 3142 50  0000 L CNN
 F 1 "Conn_01x02" H 7530 3051 50  0000 L CNN
-F 2 "Connector_Molex:Molex_Micro-Fit_3.0_43045-0200_2x01_P3.00mm_Horizontal" H 7450 3150 50  0001 C CNN
+F 2 "Connector_Molex:Molex_Micro-Fit_3.0_43045-0212_2x01_P3.00mm_Vertical" H 7450 3150 50  0001 C CNN
 F 3 "~" H 7450 3150 50  0001 C CNN
 F 4 "0430450213" H 7450 3150 50  0001 C CNN "MPN"
