File: Electronics/LCP_PowerControl/Debug.sch (KiCad schematic (older format))
At the start: 8 parts

Commit message: Aiming for rev 0.1 complete
Parts:
- J19: renamed from J?; footprint (none) -> Connector_PinSocket_2.54mm:PinSocket_1x06_P2.54mm_Vertical
- RN4: renamed from RN?; footprint (none) -> Resistor_SMD:R_Array_Concave_2x0603; MPN (none) -> EXB-V4V472JV
- gave numbers to parts that had none: 6
Connections:
- wire segments 25 -> 27
Changed lines of the file:
@@
 Sheet 11 11
 Title ""
-Date ""
-Rev ""
+Date "2020-06-17"
+Rev "R0.1"
 Comp ""
-Comment1 ""
+Comment1 "Design by: Matt Casari"
 Comment2 ""
 Comment3 ""
@@
 DEBUG_LED_2
 $Comp
-L Device:LED D?
+L Device:LED D6
 U 1 1 5EF924B3
 P 3650 4450
-F 0 "D?" V 3689 4333 50  0000 R CNN
+F 0 "D6" V 3689 4333 50  0000 R CNN
 F 1 "LED_BLUE" V 3598 4333 50  0000 R CNN
 F 2 "LED_SMD:LED_0805_2012Metric" H 3650 4450 50  0001 C CNN
@@
 $EndComp
 $Comp
-L Device:LED D?
+L Device:LED D7
 U 1 1 5EF93B88
 P 4250 4450
-F 0 "D?" V 4289 4332 50  0000 R CNN
+F 0 "D7" V 4289 4332 50  0000 R CNN
 F 1 "LED_GREEN" V 4198 4332 50  0000 R CNN
 F 2 "LED_SMD:LED_0805_2012Metric" H 4250 4450 50  0001 C CNN
@@
 $EndComp
 Wire Wire Line
-	7150 4700 4250 4700
+	7150 4700 5850 4700
 Wire Wire Line
 	4250 4700 4250 4600
@@
 	3650 4600 3650 4800
 Wire Wire Line
-	3650 4800 7150 4800
-$Comp
-L Device:R_Pack02 RN?
+	3650 4800 5400 4800
+$Comp
+L Device:R_Pack02 RN4
 U 1 1 5EF94B86
 P 4000 3800
-F 0 "RN?" H 4088 3846 50  0000 L CNN
+F 0 "RN4" H 4088 3846 50  0000 L CNN
 F 1 "R_Pack02" H 4088 3755 50  0000 L CNN
-F 2 "" V 4175 3800 50  0001 C CNN
+F 2 "Resistor_SMD:R_Array_Concave_2x0603" V 4175 3800 50  0001 C CNN
 F 3 "~" H 4000 3800 50  0001 C CNN
+F 4 "EXB-V4V472JV" H 4000 3800 50  0001 C CNN "MPN"
 	1    4000 3800
 	1    0    0    -1
 $EndComp
 $Comp
-L power:+3V3 #PWR?
+L power:+3V3 #PWR063
 U 1 1 5EF95664
 P 3950 3400
-F 0 "#PWR?" H 3950 3250 50  0001 C CNN
+F 0 "#PWR063" H 3950 3250 50  0001 C CNN
 F 1 "+3V3" H 3965 3573 50  0000 C CNN
 F 2 "" H 3950 3400 50  0001 C CNN
@@
 P 5750 3450
 AR Path="/5EE2A864/5EF976F0" Ref="J?"  Part="1"
-AR Path="/5EF8E8EB/5EF976F0" Ref="J?"  Part="1"
-F 0 "J?" H 5668 2925 50  0000 C CNN
+AR Path="/5EF8E8EB/5EF976F0" Ref="J19"  Part="1"
+F 0 "J19" H 5668 2925 50  0000 C CNN
 F 1 "Conn_01x06" H 5668 3016 50  0000 C CNN
-F 2 "" H 5750 3450 50  0001 C CNN
+F 2 "Connector_PinSocket_2.54mm:PinSocket_1x06_P2.54mm_Vertical" H 5750 3450 50  0001 C CNN
 F 3 "~" H 5750 3450 50  0001 C CNN
 	1    5750 3450
@@
 P 6200 3900
 AR Path="/5EE2A864/5EF9B9D2" Ref="#PWR?"  Part="1"
-AR Path="/5EF8E8EB/5EF9B9D2" Ref="#PWR?"  Part="1"
-F 0 "#PWR?" H 6200 3650 50  0001 C CNN
+AR Path="/5EF8E8EB/5EF9B9D2" Ref="#PWR064"  Part="1"
+F 0 "#PWR064" H 6200 3650 50  0001 C CNN
 F 1 "GND" H 6205 3727 50  0000 C CNN
 F 2 "" H 6200 3900 50  0001 C CNN
@@
 AR Path="/5EE2AB43/5EF9DADA" Ref="TP?"  Part="1"
 AR Path="/5EE7B8CC/5EF9DADA" Ref="TP?"  Part="1"
-F 0 "TP?" H 6508 3018 50  0000 L CNN
+AR Path="/5EF8E8EB/5EF9DADA" Ref="TP20"  Part="1"
+F 0 "TP20" H 6508 3018 50  0000 L CNN
 F 1 "TestPoint" H 6508 2927 50  0000 L CNN
 F 2 "TestPoint:TestPoint_Keystone_5000-5004_Miniature" H 6650 2900 50  0001 C CNN
@@
 AR Path="/5EE2AB43/5EF9DAE1" Ref="TP?"  Part="1"
 AR Path="/5EE7B8CC/5EF9DAE1" Ref="TP?"  Part="1"
-F 0 "TP?" H 6958 3018 50  0000 L CNN
+AR Path="/5EF8E8EB/5EF9DAE1" Ref="TP21"  Part="1"
+F 0 "TP21" H 6958 3018 50  0000 L CNN
 F 1 "TestPoint" H 6958 2927 50  0000 L CNN
 F 2 "TestPoint:TestPoint_Keystone_5000-5004_Miniature" H 7100 2900 50  0001 C CNN
@@
 AR Path="/5EE2AB43/5EF9E9A7" Ref="TP?"  Part="1"
 AR Path="/5EE7B8CC/5EF9E9A7" Ref="TP?"  Part="1"
-F 0 "TP?" H 5458 4618 50  0000 L CNN
+AR Path="/5EF8E8EB/5EF9E9A7" Ref="TP18"  Part="1"
+F 0 "TP18" H 5458 4618 50  0000 L CNN
 F 1 "TestPoint" H 5458 4527 50  0000 L CNN
 F 2 "TestPoint:TestPoint_Keystone_5000-5004_Miniature" H 5600 4500 50  0001 C CNN
@@
 	1    0    0    -1
 $EndComp
-Wire Wire Line
-	5400 4500 5400 4800
 $Comp
 L Connector:TestPoint TP?
@@
 AR Path="/5EE2AB43/5EF9E9AE" Ref="TP?"  Part="1"
 AR Path="/5EE7B8CC/5EF9E9AE" Ref="TP?"  Part="1"
-F 0 "TP?" H 5908 4618 50  0000 L CNN
+AR Path="/5EF8E8EB/5EF9E9AE" Ref="TP19"  Part="1"
+F 0 "TP19" H 5908 4618 50  0000 L CNN
 F 1 "TestPoint" H 5908 4527 50  0000 L CNN
 F 2 "TestPoint:TestPoint_Keystone_5000-5004_Miniature" H 6050 4500 50  0001 C CNN
@@
 $EndComp
 Wire Wire Line
+	5400 4500 5400 4800
+Connection ~ 5400 4800
+Wire Wire Line
+	5400 4800 7150 4800
+Wire Wire Line
 	5850 4500 5850 4700
+Connection ~ 5850 4700
+Wire Wire Line
+	5850 4700 4250 4700
 $EndSCHEMATC

Commit message: LCP_PowerControl Rev1
Board layout in Kicad.
Gerbers.
BOM
Parts:
- D6: MPN (none) -> APT2012LVBC/D
- D7: MPN (none) -> LTST-C171GKT
Changed lines of the file:
@@
 F 2 "LED_SMD:LED_0805_2012Metric" H 3650 4450 50  0001 C CNN
 F 3 "~" H 3650 4450 50  0001 C CNN
+F 4 "APT2012LVBC/D" V 3650 4450 50  0001 C CNN "MPN"
 	1    3650 4450
 	0    -1   -1   0
@@
 F 2 "LED_SMD:LED_0805_2012Metric" H 4250 4450 50  0001 C CNN
 F 3 "~" H 4250 4450 50  0001 C CNN
+F 4 "LTST-C171GKT" V 4250 4450 50  0001 C CNN "MPN"
 	1    4250 4450
 	0    -1   -1   0

Commit message: Rev1
Removed test points. Cleaned up unnecessary traces. Fixed electrical issues #1-#7
Parts:
- removed TP18, TP19, TP20, TP21: TestPoint, TestPoint:TestPoint_Keystone_5000-5004_Miniature, symbol Connector:TestPoint
Changed lines of the file:
@@
 $EndComp
-Wire Wire Line
-	7150 4700 5850 4700
 Wire Wire Line
 	4250 4700 4250 4600
 Wire Wire Line
 	3650 4600 3650 4800
-Wire Wire Line
-	3650 4800 5400 4800
 $Comp
 L Device:R_Pack02 RN4
@@
 	-1   0    0    1
 $EndComp
-Wire Wire Line
-	7150 3250 6900 3250
-Wire Wire Line
-	5950 3350 6450 3350
 $Comp
 L power:GND #PWR?
@@
 NoConn ~ 5950 3450
 NoConn ~ 5950 3550
-$Comp
-L Connector:TestPoint TP?
-U 1 1 5EF9DADA
-P 6450 2900
-AR Path="/5EE2AB43/5EF9DADA" Ref="TP?"  Part="1"
-AR Path="/5EE7B8CC/5EF9DADA" Ref="TP?"  Part="1"
-AR Path="/5EF8E8EB/5EF9DADA" Ref="TP20"  Part="1"
-F 0 "TP20" H 6508 3018 50  0000 L CNN
-F 1 "TestPoint" H 6508 2927 50  0000 L CNN
-F 2 "TestPoint:TestPoint_Keystone_5000-5004_Miniature" H 6650 2900 50  0001 C CNN
-F 3 "~" H 6650 2900 50  0001 C CNN
-	1    6450 2900
-	1    0    0    -1
-$EndComp
-$Comp
-L Connector:TestPoint TP?
-U 1 1 5EF9DAE1
-P 6900 2900
-AR Path="/5EE2AB43/5EF9DAE1" Ref="TP?"  Part="1"
-AR Path="/5EE7B8CC/5EF9DAE1" Ref="TP?"  Part="1"
-AR Path="/5EF8E8EB/5EF9DAE1" Ref="TP21"  Part="1"
-F 0 "TP21" H 6958 3018 50  0000 L CNN
-F 1 "TestPoint" H 6958 2927 50  0000 L CNN
-F 2 "TestPoint:TestPoint_Keystone_5000-5004_Miniature" H 7100 2900 50  0001 C CNN
-F 3 "~" H 7100 2900 50  0001 C CNN
-	1    6900 2900
-	1    0    0    -1
-$EndComp
 Wire Wire Line
-	6900 2900 6900 3250
-Connection ~ 6900 3250
+	3650 4800 7150 4800
 Wire Wire Line
-	6900 3250 5950 3250
+	4250 4700 7150 4700
 Wire Wire Line
-	6450 2900 6450 3350
-Connection ~ 6450 3350
+	5950 3250 7150 3250
 Wire Wire Line
-	6450 3350 7150 3350
-$Comp
-L Connector:TestPoint TP?
-U 1 1 5EF9E9A7
-P 5400 4500
-AR Path="/5EE2AB43/5EF9E9A7" Ref="TP?"  Part="1"
-AR Path="/5EE7B8CC/5EF9E9A7" Ref="TP?"  Part="1"
-AR Path="/5EF8E8EB/5EF9E9A7" Ref="TP18"  Part="1"
-F 0 "TP18" H 5458 4618 50  0000 L CNN
-F 1 "TestPoint" H 5458 4527 50  0000 L CNN
-F 2 "TestPoint:TestPoint_Keystone_5000-5004_Miniature" H 5600 4500 50  0001 C CNN
-F 3 "~" H 5600 4500 50  0001 C CNN
-	1    5400 4500
-	1    0    0    -1
-$EndComp
-$Comp
-L Connector:TestPoint TP?
-U 1 1 5EF9E9AE
-P 5850 4500
-AR Path="/5EE2AB43/5EF9E9AE" Ref="TP?"  Part="1"
-AR Path="/5EE7B8CC/5EF9E9AE" Ref="TP?"  Part="1"
-AR Path="/5EF8E8EB/5EF9E9AE" Ref="TP19"  Part="1"
-F 0 "TP19" H 5908 4618 50  0000 L CNN
-F 1 "TestPoint" H 5908 4527 50  0000 L CNN
-F 2 "TestPoint:TestPoint_Keystone_5000-5004_Miniature" H 6050 4500 50  0001 C CNN
-F 3 "~" H 6050 4500 50  0001 C CNN
-	1    5850 4500
-	1    0    0    -1
-$EndComp
-Wire Wire Line
-	5400 4500 5400 4800
-Connection ~ 5400 4800
-Wire Wire Line
-	5400 4800 7150 4800
-Wire Wire Line
-	5850 4500 5850 4700
-Connection ~ 5850 4700
-Wire Wire Line
-	5850 4700 4250 4700
+	5950 3350 7150 3350
 $EndSCHEMATC

Commit message: BOM Update
Updated MPNs on components to match supplies as well as correcting some resistor values
Parts:
- J19: MPN (none) -> 61300611121
Changed lines of the file:
@@
 F 2 "Connector_PinSocket_2.54mm:PinSocket_1x06_P2.54mm_Vertical" H 5750 3450 50  0001 C CNN
 F 3 "~" H 5750 3450 50  0001 C CNN
+F 4 "61300611121" H 5750 3450 50  0001 C CNN "MPN"
 	1    5750 3450
 	-1   0    0    1

Commit message: Rev 1 Update
Issues #9-#13 fixed
Rev 1 Gerbers & BOM Ready
Parts:
- removed J19: Conn_01x06, Connector_PinSocket_2.54mm:PinSocket_1x06_P2.54mm_Vertical, symbol Connector_Generic:Conn_01x06
- D7: MPN LTST-C171GKT -> APT2012SGC
Connections:
- no-connect marks 3 -> 0
Changed lines of the file:
@@
 Comment4 ""
 $EndDescr
-Text HLabel 7150 3350 2    50   Input ~ 0
-DEBUG_TX
-Text HLabel 7150 3250 2    50   Output ~ 0
-DEBUG_RX
 Text HLabel 7150 4700 2    50   Input ~ 0
 DEBUG_LED_1
@@
 F 2 "LED_SMD:LED_0805_2012Metric" H 4250 4450 50  0001 C CNN
 F 3 "~" H 4250 4450 50  0001 C CNN
-F 4 "LTST-C171GKT" V 4250 4450 50  0001 C CNN "MPN"
+F 4 "APT2012SGC" V 4250 4450 50  0001 C CNN "MPN"
 	1    4250 4450
 	0    -1   -1   0
@@
 Wire Wire Line
 	4000 4150 4000 4000
-$Comp
-L Connector_Generic:Conn_01x06 J?
-U 1 1 5EF976F0
-P 5750 3450
-AR Path="/5EE2A864/5EF976F0" Ref="J?"  Part="1"
-AR Path="/5EF8E8EB/5EF976F0" Ref="J19"  Part="1"
-F 0 "J19" H 5668 2925 50  0000 C CNN
-F 1 "Conn_01x06" H 5668 3016 50  0000 C CNN
-F 2 "Connector_PinSocket_2.54mm:PinSocket_1x06_P2.54mm_Vertical" H 5750 3450 50  0001 C CNN
-F 3 "~" H 5750 3450 50  0001 C CNN
-F 4 "61300611121" H 5750 3450 50  0001 C CNN "MPN"
-	1    5750 3450
-	-1   0    0    1
-$EndComp
-$Comp
-L power:GND #PWR?
-U 1 1 5EF9B9D2
-P 6200 3900
-AR Path="/5EE2A864/5EF9B9D2" Ref="#PWR?"  Part="1"
-AR Path="/5EF8E8EB/5EF9B9D2" Ref="#PWR064"  Part="1"
-F 0 "#PWR064" H 6200 3650 50  0001 C CNN
-F 1 "GND" H 6205 3727 50  0000 C CNN
-F 2 "" H 6200 3900 50  0001 C CNN
-F 3 "" H 6200 3900 50  0001 C CNN
-	1    6200 3900
-	1    0    0    -1
-$EndComp
-Wire Wire Line
-	5950 3650 6200 3650
-Wire Wire Line
-	6200 3650 6200 3900
-NoConn ~ 5950 3150
-NoConn ~ 5950 3450
-NoConn ~ 5950 3550
 Wire Wire Line
 	3650 4800 7150 4800
 Wire Wire Line
 	4250 4700 7150 4700
-Wire Wire Line
-	5950 3250 7150 3250
-Wire Wire Line
-	5950 3350 7150 3350
 $EndSCHEMATC

Commit message: LCP PowerControl Board Update
Parts:
- RN4: value R_Pack02 -> 4.7k
Changed lines of the file:
@@
 P 4000 3800
 F 0 "RN4" H 4088 3846 50  0000 L CNN
-F 1 "R_Pack02" H 4088 3755 50  0000 L CNN
+F 1 "4.7k" H 4088 3755 50  0000 L CNN
 F 2 "Resistor_SMD:R_Array_Concave_2x0603" V 4175 3800 50  0001 C CNN
 F 3 "~" H 4000 3800 50  0001 C CNN
