File: Electronics/LCP_PowerControl/PowerMonitoring.sch (KiCad schematic (older format))
At the start: 18 parts, among them Q2 2N7002, U1 MAX17205

Commit message: LCP PowerControl Board Update
Parts:
- C1: MPN CL31B105KCHNNNE -> GCM21BC72A105KE36L
- D1, D2, D3, D4: MPN SZMM3Z5V6ST1G -> UDZ5V6B-7
- Q2, e1: value 2N7002 -> ZVN4106FTA; MPN 2N7002-7-F -> ZVN4106FTA
Changed lines of the file:
@@
 P 3800 3600
 F 0 "e1" H 4005 3646 50  0000 L CNN
-F 1 "2N7002" H 4005 3555 50  0000 L CNN
+F 1 "ZVN4106FTA" H 4005 3555 50  0000 L CNN
 F 2 "Package_TO_SOT_SMD:SOT-23" H 4000 3525 50  0001 L CIN
 F 3 "https://www.fairchildsemi.com/datasheets/2N/2N7002.pdf" H 3800 3600 50  0001 L CNN
-F 4 "2N7002-7-F" H 3800 3600 50  0001 C CNN "MPN"
+F 4 "ZVN4106FTA" H 3800 3600 50  0001 C CNN "MPN"
 	1    3800 3600
 	-1   0    0    -1
@@
 F 2 "Diode_SMD:D_SOD-323_HandSoldering" H 7950 4000 50  0001 C CNN
 F 3 "~" H 7950 4000 50  0001 C CNN
-F 4 "SZMM3Z5V6ST1G" V 7950 4000 50  0001 C CNN "MPN"
+F 4 "UDZ5V6B-7" V 7950 4000 50  0001 C CNN "MPN"
 	1    7950 4000
 	0    1    1    0
@@
 F 2 "Diode_SMD:D_SOD-323_HandSoldering" H 7650 4000 50  0001 C CNN
 F 3 "~" H 7650 4000 50  0001 C CNN
-F 4 "SZMM3Z5V6ST1G" V 7650 4000 50  0001 C CNN "MPN"
+F 4 "UDZ5V6B-7" V 7650 4000 50  0001 C CNN "MPN"
 	1    7650 4000
 	0    1    1    0
@@
 F 2 "Diode_SMD:D_SOD-323_HandSoldering" H 8250 4000 50  0001 C CNN
 F 3 "~" H 8250 4000 50  0001 C CNN
-F 4 "SZMM3Z5V6ST1G" V 8250 4000 50  0001 C CNN "MPN"
+F 4 "UDZ5V6B-7" V 8250 4000 50  0001 C CNN "MPN"
 	1    8250 4000
 	0    1    1    0
@@
 P 4800 2750
 F 0 "Q2" H 5004 2796 50  0000 L CNN
-F 1 "2N7002" H 5004 2705 50  0000 L CNN
+F 1 "ZVN4106FTA" H 5004 2705 50  0000 L CNN
 F 2 "Package_TO_SOT_SMD:SOT-23" H 5000 2675 50  0001 L CIN
 F 3 "https://www.fairchildsemi.com/datasheets/2N/2N7002.pdf" H 4800 2750 50  0001 L CNN
-F 4 "2N7002-7-F" H 4800 2750 50  0001 C CNN "MPN"
+F 4 "ZVN4106FTA" H 4800 2750 50  0001 C CNN "MPN"
 	1    4800 2750
 	1    0    0    -1
@@
 F 2 "Diode_SMD:D_SOD-323_HandSoldering" H 4350 3000 50  0001 C CNN
 F 3 "~" H 4350 3000 50  0001 C CNN
-F 4 "SZMM3Z5V6ST1G" V 4350 3000 50  0001 C CNN "MPN"
+F 4 "UDZ5V6B-7" V 4350 3000 50  0001 C CNN "MPN"
 	1    4350 3000
 	0    1    1    0
@@
 F 2 "Capacitor_SMD:C_0805_2012Metric" H 4938 3000 50  0001 C CNN
 F 3 "~" H 4900 3150 50  0001 C CNN
-F 4 "CL31B105KCHNNNE" H 4900 3150 50  0001 C CNN "MPN"
+F 4 "GCM21BC72A105KE36L" H 4900 3150 50  0001 C CNN "MPN"
 	1    4900 3150
 	1    0    0    -1
