File: Electronics/LCP_PowerControl/PowerRegulators.sch (KiCad schematic (older format))
At the start: 0 parts

Commit message: Adding libraries and recent changes
Parts:
- added C?: 1uF, Capacitor_SMD:C_0603_1608Metric, symbol Device:C
- added C?: 0.1uF, Capacitor_SMD:C_0603_1608Metric, symbol Device:C
- added C?: 0.1uF, Capacitor_SMD:C_0402_1005Metric, symbol Device:C
- added C? (x2): 10uF, Capacitor_SMD:C_1206_3216Metric, symbol Device:C
- added L?: L, symbol Device:L
- added R?: 51k, Resistor_SMD:R_0603_1608Metric, symbol Device:R
- added R?: 22.1k, Resistor_SMD:R_0402_1005Metric, symbol Device:R
- added TP? (x9): TestPoint, TestPoint:TestPoint_Keystone_5000-5004_Miniature, symbol Connector:TestPoint
- added U?: LMR50410, Package_TO_SOT_SMD:SOT-23-6_Handsoldering, symbol PMEL_PowerICs:LMR50410
Connections:
- new net: C?.2, R?.1, R?.2, U?.1 (CB)
- new net: C?.1, L?.1, U?.6 (SW)
- new net +12V: TP?.1
- new net +3V3: C?.1, C?.1, L?.2, R?.1, TP?.1, TP?.1
- new net +BATT: C?.1, C?.1, TP?.1, U?.4 (EN), U?.5 (VIN)
- new net GND: C?.2, C?.2, C?.2, C?.2, R?.2, TP?.1, TP?.1, TP?.1, TP?.1, U?.2 (GND)
Other:
- note added: "12V Regulator"
- note added: "3V3 Regulator"

Commit message: Aiming for rev 0.1 complete
Parts:
- added C17, C18, C23, C25: 10uF, Capacitor_SMD:C_1210_3225Metric, symbol Device:C
- added C20, C22: 0.22uF, Capacitor_SMD:C_0603_1608Metric, symbol Device:C
- added C24: 1.0uF, Capacitor_SMD:C_0603_1608Metric, symbol Device:C
- added C27: 0.1uF, Capacitor_SMD:C_0402_1005Metric, symbol Device:C
- added C30: DNP, Capacitor_SMD:C_0603_1608Metric, symbol Device:C
- added C31, C32, C33: 10uF, Resistor_SMD:R_0603_1608Metric, symbol Device:C
- added L2: 10uH, symbol Device:L
- added R14: 26.7k, Resistor_SMD:R_0402_1005Metric, symbol Device:R
- added R15, R18: 100k, Resistor_SMD:R_0402_1005Metric, symbol Device:R
- added R19: 9.09k, Resistor_SMD:R_0402_1005Metric, symbol Device:R
- added R20: 1k, Resistor_SMD:R_0402_1005Metric, symbol Device:R
- added U5: LM61460, symbol PMEL_PowerICs:LM61460
- L1: renamed from L?; value L -> 12uH; MPN (none) -> SDR0805-120ML
- gave numbers to parts that had none: 17
Connections:
- net +12V: now also C30.1, C31.1, C32.1, C33.1, L2.2, R15.2, R18.2, U5.1 (BIAS)
- net +BATT: now also C17.1, C18.1, C20.1, C22.1, C23.1, C25.1, U5.12 (VIN2), U5.8 (VIN1)
- net 12V_ENABLE: now also TP13.1, U5.7 (EN/SYNC)
- net GND: now also C17.2, C18.2, C20.2, C22.2, C23.2, C24.2, C25.2, C31.2, C32.2, C33.2, R14.2, R19.1, U5.11 (PGND2), U5.3 (AGND), U5.9 (PGND1)
- net at C26.2, U4.1 (CB): no longer R16.2, R17.1
- net at U4.3 (FB): now also R16.2, R17.1
- new net: C27.2, L2.1, U5.10 (SW)
- new net: C24.1, U5.2 (VCC)
- new net: C30.2, R20.2
- new net: C27.1, U5.13 (RBOOT), U5.14 (CBOOT)
- new net: R14.1, U5.6 (RT)
- new net: R18.1, R19.2, R20.1, U5.4 (FB)
- new net: R15.1, U5.5 (PGOOD)
Other:
- moved on the sheet: TP10, TP11, TP12, TP13, TP14, TP15, TP7, TP8, TP9

Commit message: KiCad Layout
Component and Traces finished. Need a look over. Will work on Silkscreen
after.

JTAG Connector. Should pin 1 be pulled up w/ 470Ohm resistor similar to
other designs? Also TDI and TMI signals are connected, is this correct?
Parts:
- L1: footprint (none) -> Inductor_SMD:L_Bourns-SRN8040_8x8.15mm
- L2: footprint (none) -> Inductor_SMD:L_Coilcraft_XAL1010
- U5: footprint (none) -> Converter_DCDC:TI_RJR0014A
Changed lines of the file:
@@
 F 0 "L1" V 6940 1850 50  0000 C CNN
 F 1 "12uH" V 6849 1850 50  0000 C CNN
-F 2 "" H 6750 1850 50  0001 C CNN
+F 2 "Inductor_SMD:L_Bourns-SRN8040_8x8.15mm" H 6750 1850 50  0001 C CNN
 F 3 "~" H 6750 1850 50  0001 C CNN
 F 4 "SDR0805-120ML" H 6750 1850 50  0001 C CNN "MPN"
@@
 F 0 "L2" V 7190 5050 50  0000 C CNN
 F 1 "10uH" V 7099 5050 50  0000 C CNN
-F 2 "" H 7000 5050 50  0001 C CNN
+F 2 "Inductor_SMD:L_Coilcraft_XAL1010" H 7000 5050 50  0001 C CNN
 F 3 "http://www.coilcraft.com/pdfs/xal1010.pdf" H 7000 5050 50  0001 C CNN
 F 4 "XAL1010-103MEB" V 7000 5050 50  0001 C CNN "MPN"
@@
 F 0 "U5" H 6050 6000 50  0000 C CNN
 F 1 "LM61460" H 5500 6000 50  0000 C CNN
-F 2 "" H 5200 6400 50  0001 C CNN
+F 2 "Converter_DCDC:TI_RJR0014A" H 5200 6400 50  0001 C CNN
 F 3 "https://www.ti.com/lit/ds/symlink/lm61460-q1.pdf?ts=1592411830672&ref_url=https%253A%252F%252Fwww.ti.com%252Fproduct%252FLM61460-Q1" H 5200 6400 50  0001 C CNN
 	1    5800 5200

Commit message: LCP_PowerControl Rev1
Board layout in Kicad.
Gerbers.
BOM
Parts:
- C19: MPN (none) -> C1206X7R101-105KNE
- C21: MPN (none) -> GCM188R71H104KA57J
- C26: MPN (none) -> GRM155R71A104KA01D
- C28, C29: MPN (none) -> CL31B106KPHVPNE
- R16: MPN (none) -> MCT0603C5102FP500
- R17: MPN (none) -> RMCF0402FT22K1
- U4: MPN (none) -> LMR50410YQDBVRQ1
- U5: MPN (none) -> LM61460AANRJRR
Changed lines of the file:
@@
 F 2 "Package_TO_SOT_SMD:SOT-23-6_Handsoldering" H 5150 1650 50  0001 C CNN
 F 3 "https://www.ti.com/lit/ds/symlink/lmr50410.pdf?ts=1591402847494&ref_url=https://www.ti.com/product/LMR50410" H 5050 2100 50  0001 C CNN
+F 4 "LMR50410YQDBVRQ1" H 5200 1950 50  0001 C CNN "MPN"
 	1    5200 1950
 	1    0    0    -1
@@
 F 2 "Capacitor_SMD:C_0603_1608Metric" H 3338 1950 50  0001 C CNN
 F 3 "~" H 3300 2100 50  0001 C CNN
+F 4 "C1206X7R101-105KNE" H 3300 2100 50  0001 C CNN "MPN"
 	1    3300 2100
 	1    0    0    -1
@@
 F 2 "Capacitor_SMD:C_0603_1608Metric" H 3688 1950 50  0001 C CNN
 F 3 "~" H 3650 2100 50  0001 C CNN
+F 4 "GCM188R71H104KA57J" H 3650 2100 50  0001 C CNN "MPN"
 	1    3650 2100
 	1    0    0    -1
@@
 F 2 "Capacitor_SMD:C_0402_1005Metric" H 6465 1959 50  0001 L CNN
 F 3 "~" H 6350 2050 50  0001 C CNN
+F 4 "GRM155R71A104KA01D" H 6350 2050 50  0001 C CNN "MPN"
 	1    6350 2050
 	1    0    0    -1
@@
 F 2 "Capacitor_SMD:C_1206_3216Metric" H 7788 1900 50  0001 C CNN
 F 3 "~" H 7750 2050 50  0001 C CNN
+F 4 "CL31B106KPHVPNE" H 7750 2050 50  0001 C CNN "MPN"
 	1    7750 2050
 	1    0    0    -1
@@
 F 2 "Capacitor_SMD:C_1206_3216Metric" H 8188 1900 50  0001 C CNN
 F 3 "~" H 8150 2050 50  0001 C CNN
+F 4 "CL31B106KPHVPNE" H 8150 2050 50  0001 C CNN "MPN"
 	1    8150 2050
 	1    0    0    -1
@@
 F 2 "Resistor_SMD:R_0603_1608Metric" V 6980 2150 50  0001 C CNN
 F 3 "~" H 7050 2150 50  0001 C CNN
+F 4 "MCT0603C5102FP500" H 7050 2150 50  0001 C CNN "MPN"
 	1    7050 2150
 	1    0    0    -1
@@
 F 2 "Resistor_SMD:R_0402_1005Metric" V 6980 2650 50  0001 C CNN
 F 3 "~" H 7050 2650 50  0001 C CNN
+F 4 "RMCF0402FT22K1" H 7050 2650 50  0001 C CNN "MPN"
 	1    7050 2650
 	1    0    0    -1
@@
 F 2 "Converter_DCDC:TI_RJR0014A" H 5200 6400 50  0001 C CNN
 F 3 "https://www.ti.com/lit/ds/symlink/lm61460-q1.pdf?ts=1592411830672&ref_url=https%253A%252F%252Fwww.ti.com%252Fproduct%252FLM61460-Q1" H 5200 6400 50  0001 C CNN
+F 4 "LM61460AANRJRR" H 5800 5200 50  0001 C CNN "MPN"
 	1    5800 5200
 	1    0    0    -1

Commit message: Rev1
Removed test points. Cleaned up unnecessary traces. Fixed electrical issues #1-#7
Parts:
- removed TP10, TP12, TP14, TP15: TestPoint, TestPoint:TestPoint_Keystone_5000-5004_Miniature, symbol Connector:TestPoint
Changed lines of the file:
@@
-$EndComp
-$Comp
-L Connector:TestPoint TP?
-U 1 1 5EE9902D
-P 2400 6450
-AR Path="/5EE2A7AF/5EE9902D" Ref="TP?"  Part="1"
-AR Path="/5EE4388C/5EE9902D" Ref="TP14"  Part="1"
-F 0 "TP14" H 2458 6568 50  0000 L CNN
-F 1 "TestPoint" H 2458 6477 50  0000 L CNN
-F 2 "TestPoint:TestPoint_Keystone_5000-5004_Miniature" H 2600 6450 50  0001 C CNN
-F 3 "~" H 2600 6450 50  0001 C CNN
-F 4 "5000" H 2400 6450 50  0001 C CNN "MPN"
-	1    2400 6450
-	1    0    0    -1
 $EndComp
 $Comp
@@
 $EndComp
 $Comp
-L Connector:TestPoint TP10
-U 1 1 5EE9A55C
-P 1500 7200
-F 0 "TP10" H 1558 7318 50  0000 L CNN
-F 1 "TestPoint" H 1558 7227 50  0000 L CNN
-F 2 "TestPoint:TestPoint_Keystone_5000-5004_Miniature" H 1700 7200 50  0001 C CNN
-F 3 "~" H 1700 7200 50  0001 C CNN
-F 4 "5001" H 1500 7200 50  0001 C CNN "MPN"
-	1    1500 7200
-	1    0    0    -1
-$EndComp
-$Comp
-L Connector:TestPoint TP12
-U 1 1 5EE9A563
-P 1950 7200
-F 0 "TP12" H 2008 7318 50  0000 L CNN
-F 1 "TestPoint" H 2008 7227 50  0000 L CNN
-F 2 "TestPoint:TestPoint_Keystone_5000-5004_Miniature" H 2150 7200 50  0001 C CNN
-F 3 "~" H 2150 7200 50  0001 C CNN
-F 4 "5001" H 1950 7200 50  0001 C CNN "MPN"
-	1    1950 7200
-	1    0    0    -1
-$EndComp
-$Comp
-L Connector:TestPoint TP15
-U 1 1 5EE9A56A
-P 2400 7200
-F 0 "TP15" H 2458 7318 50  0000 L CNN
-F 1 "TestPoint" H 2458 7227 50  0000 L CNN
-F 2 "TestPoint:TestPoint_Keystone_5000-5004_Miniature" H 2600 7200 50  0001 C CNN
-F 3 "~" H 2600 7200 50  0001 C CNN
-F 4 "5001" H 2400 7200 50  0001 C CNN "MPN"
-	1    2400 7200
-	1    0    0    -1
-$EndComp
-$Comp
 L power:GND #PWR037
 U 1 1 5EE9D7F2
@@
 	1    0    0    -1
 $EndComp
-$Comp
-L power:GND #PWR040
-U 1 1 5EE9DD4E
-P 1500 7350
-F 0 "#PWR040" H 1500 7100 50  0001 C CNN
-F 1 "GND" H 1505 7177 50  0000 C CNN
-F 2 "" H 1500 7350 50  0001 C CNN
-F 3 "" H 1500 7350 50  0001 C CNN
-	1    1500 7350
-	1    0    0    -1
-$EndComp
-$Comp
-L power:GND #PWR042
-U 1 1 5EE9DFE6
-P 1950 7350
-F 0 "#PWR042" H 1950 7100 50  0001 C CNN
-F 1 "GND" H 1955 7177 50  0000 C CNN
-F 2 "" H 1950 7350 50  0001 C CNN
-F 3 "" H 1950 7350 50  0001 C CNN
-	1    1950 7350
-	1    0    0    -1
-$EndComp
-$Comp
-L power:GND #PWR044
-U 1 1 5EE9E1B5
-P 2400 7350
-F 0 "#PWR044" H 2400 7100 50  0001 C CNN
-F 1 "GND" H 2405 7177 50  0000 C CNN
-F 2 "" H 2400 7350 50  0001 C CNN
-F 3 "" H 2400 7350 50  0001 C CNN
-	1    2400 7350
-	1    0    0    -1
-$EndComp
-Wire Wire Line
-	2400 7200 2400 7350
-Wire Wire Line
-	1950 7200 1950 7350
-Wire Wire Line
-	1500 7200 1500 7350
 Wire Wire Line
 	1000 7200 1000 7350
-$Comp
-L power:+3V3 #PWR045
-U 1 1 5EEA0E5C
-P 2550 6700
-F 0 "#PWR045" H 2550 6550 50  0001 C CNN
-F 1 "+3V3" H 2565 6873 50  0000 C CNN
-F 2 "" H 2550 6700 50  0001 C CNN
-F 3 "" H 2550 6700 50  0001 C CNN
-	1    2550 6700
-	1    0    0    -1
-$EndComp
 $Comp
 L power:+12V #PWR041
@@
 Wire Wire Line
 	2100 6800 2100 6700
-Wire Wire Line
-	2400 6450 2400 6800
-Wire Wire Line
-	2400 6800 2550 6800
-Wire Wire Line
-	2550 6800 2550 6700
 $Comp
 L Device:L L2

Commit message: BOM Update
Updated MPNs on components to match supplies as well as correcting some resistor values
Parts:
- C19: MPN C1206X7R101-105KNE -> CL10A105KB8NNNC
- C31, C32, C33: MPN C3225X7R1H106M250AC -> CL10A106MA8NRNC
- R16: MPN MCT0603C5102FP500 -> RC0603FR-0751KL
- TP11, TP7, TP9: MPN 5000 -> (none)
- TP13, TP8: MPN 5001 -> (none)
Changed lines of the file:
@@
 F 2 "Capacitor_SMD:C_0603_1608Metric" H 3338 1950 50  0001 C CNN
 F 3 "~" H 3300 2100 50  0001 C CNN
-F 4 "C1206X7R101-105KNE" H 3300 2100 50  0001 C CNN "MPN"
+F 4 "CL10A105KB8NNNC" H 3300 2100 50  0001 C CNN "MPN"
 	1    3300 2100
 	1    0    0    -1
@@
 F 2 "Resistor_SMD:R_0603_1608Metric" V 6980 2150 50  0001 C CNN
 F 3 "~" H 7050 2150 50  0001 C CNN
-F 4 "MCT0603C5102FP500" H 7050 2150 50  0001 C CNN "MPN"
+F 4 "RC0603FR-0751KL" H 7050 2150 50  0001 C CNN "MPN"
 	1    7050 2150
 	1    0    0    -1
@@
 F 2 "TestPoint:TestPoint_Keystone_5000-5004_Miniature" H 1200 6450 50  0001 C CNN
 F 3 "~" H 1200 6450 50  0001 C CNN
-F 4 "5000" H 1000 6450 50  0001 C CNN "MPN"
+F 4 "" H 1000 6450 50  0001 C CNN "MPN"
 	1    1000 6450
 	1    0    0    -1
@@
 F 2 "TestPoint:TestPoint_Keystone_5000-5004_Miniature" H 2200 5050 50  0001 C CNN
 F 3 "~" H 2200 5050 50  0001 C CNN
-F 4 "5001" H 2000 5050 50  0001 C CNN "MPN"
+F 4 "" H 2000 5050 50  0001 C CNN "MPN"
 	1    2000 5050
 	1    0    0    -1
@@
 F 2 "TestPoint:TestPoint_Keystone_5000-5004_Miniature" H 1700 6450 50  0001 C CNN
 F 3 "~" H 1700 6450 50  0001 C CNN
-F 4 "5000" H 1500 6450 50  0001 C CNN "MPN"
+F 4 "" H 1500 6450 50  0001 C CNN "MPN"
 	1    1500 6450
 	1    0    0    -1
@@
 F 2 "TestPoint:TestPoint_Keystone_5000-5004_Miniature" H 2150 6450 50  0001 C CNN
 F 3 "~" H 2150 6450 50  0001 C CNN
-F 4 "5000" H 1950 6450 50  0001 C CNN "MPN"
+F 4 "" H 1950 6450 50  0001 C CNN "MPN"
 	1    1950 6450
 	1    0    0    -1
@@
 F 2 "TestPoint:TestPoint_Keystone_5000-5004_Miniature" H 1200 7200 50  0001 C CNN
 F 3 "~" H 1200 7200 50  0001 C CNN
-F 4 "5001" H 1000 7200 50  0001 C CNN "MPN"
+F 4 "" H 1000 7200 50  0001 C CNN "MPN"
 	1    1000 7200
 	1    0    0    -1
@@
 F 2 "Resistor_SMD:R_0603_1608Metric" H 9738 5150 50  0001 C CNN
 F 3 "~" H 9700 5300 50  0001 C CNN
-F 4 "C3225X7R1H106M250AC" H 9700 5300 50  0001 C CNN "MPN"
+F 4 "CL10A106MA8NRNC" H 9700 5300 50  0001 C CNN "MPN"
 	1    9700 5300
 	1    0    0    -1
@@
 F 2 "Resistor_SMD:R_0603_1608Metric" H 10138 5150 50  0001 C CNN
 F 3 "~" H 10100 5300 50  0001 C CNN
-F 4 "C3225X7R1H106M250AC" H 10100 5300 50  0001 C CNN "MPN"
+F 4 "CL10A106MA8NRNC" H 10100 5300 50  0001 C CNN "MPN"
 	1    10100 5300
 	1    0    0    -1
@@
 F 2 "Resistor_SMD:R_0603_1608Metric" H 10538 5150 50  0001 C CNN
 F 3 "~" H 10500 5300 50  0001 C CNN
-F 4 "C3225X7R1H106M250AC" H 10500 5300 50  0001 C CNN "MPN"
+F 4 "CL10A106MA8NRNC" H 10500 5300 50  0001 C CNN "MPN"
 	1    10500 5300
 	1    0    0    -1

Commit message: Rev 1 Update
Issues #9-#13 fixed
Rev 1 Gerbers & BOM Ready
Parts:
- C20, C22: MPN CGA3E3X7R1H224K080AB -> C1608X7R1H224K080AE
- C31, C32, C33: MPN CL10A106MA8NRNC -> C1608X5R1E106M080AC
- R15, R18: MPN CRCW0402100KFKED -> RMCF0402FT100K
- R20: MPN CRCW04021K00FKED -> PFR05S-102-FNH
- U5: MPN LM61460AANRJRR -> LMQ61460AFSQRJRRQ1
Changed lines of the file:
@@
 F 2 "Capacitor_SMD:C_0603_1608Metric" H 4038 4100 50  0001 C CNN
 F 3 "~" H 4000 4250 50  0001 C CNN
-F 4 "CGA3E3X7R1H224K080AB" H 4000 4250 50  0001 C CNN "MPN"
+F 4 "C1608X7R1H224K080AE" H 4000 4250 50  0001 C CNN "MPN"
 	1    4000 4250
 	1    0    0    -1
@@
 F 2 "Resistor_SMD:R_0402_1005Metric" V 8430 5300 50  0001 C CNN
 F 3 "~" H 8500 5300 50  0001 C CNN
-F 4 "CRCW0402100KFKED" H 8500 5300 50  0001 C CNN "MPN"
+F 4 "RMCF0402FT100K" H 8500 5300 50  0001 C CNN "MPN"
 	1    8500 5300
 	-1   0    0    1
@@
 F 2 "Resistor_SMD:R_0402_1005Metric" V 8830 5500 50  0001 C CNN
 F 3 "~" H 8900 5500 50  0001 C CNN
-F 4 "CRCW04021K00FKED" V 8900 5500 50  0001 C CNN "MPN"
+F 4 "PFR05S-102-FNH" V 8900 5500 50  0001 C CNN "MPN"
 	1    8900 5500
 	0    -1   -1   0
@@
 F 2 "Resistor_SMD:R_0603_1608Metric" H 9738 5150 50  0001 C CNN
 F 3 "~" H 9700 5300 50  0001 C CNN
-F 4 "CL10A106MA8NRNC" H 9700 5300 50  0001 C CNN "MPN"
+F 4 "C1608X5R1E106M080AC" H 9700 5300 50  0001 C CNN "MPN"
 	1    9700 5300
 	1    0    0    -1
@@
 F 2 "Capacitor_SMD:C_0603_1608Metric" H 3538 4100 50  0001 C CNN
 F 3 "~" H 3500 4250 50  0001 C CNN
-F 4 "CGA3E3X7R1H224K080AB" H 3500 4250 50  0001 C CNN "MPN"
+F 4 "C1608X7R1H224K080AE" H 3500 4250 50  0001 C CNN "MPN"
 	1    3500 4250
 	1    0    0    -1
@@
 F 2 "Resistor_SMD:R_0402_1005Metric" V 5730 6400 50  0001 C CNN
 F 3 "~" H 5800 6400 50  0001 C CNN
-F 4 "CRCW0402100KFKED" H 5800 6400 50  0001 C CNN "MPN"
+F 4 "RMCF0402FT100K" H 5800 6400 50  0001 C CNN "MPN"
 	1    5800 6400
 	0    -1   -1   0
@@
 F 2 "Resistor_SMD:R_0603_1608Metric" H 10138 5150 50  0001 C CNN
 F 3 "~" H 10100 5300 50  0001 C CNN
-F 4 "CL10A106MA8NRNC" H 10100 5300 50  0001 C CNN "MPN"
+F 4 "C1608X5R1E106M080AC" H 10100 5300 50  0001 C CNN "MPN"
 	1    10100 5300
 	1    0    0    -1
@@
 F 2 "Resistor_SMD:R_0603_1608Metric" H 10538 5150 50  0001 C CNN
 F 3 "~" H 10500 5300 50  0001 C CNN
-F 4 "CL10A106MA8NRNC" H 10500 5300 50  0001 C CNN "MPN"
+F 4 "C1608X5R1E106M080AC" H 10500 5300 50  0001 C CNN "MPN"
 	1    10500 5300
 	1    0    0    -1
@@
 F 2 "Converter_DCDC:TI_RJR0014A" H 5200 6400 50  0001 C CNN
 F 3 "https://www.ti.com/lit/ds/symlink/lm61460-q1.pdf?ts=1592411830672&ref_url=https%253A%252F%252Fwww.ti.com%252Fproduct%252FLM61460-Q1" H 5200 6400 50  0001 C CNN
-F 4 "LM61460AANRJRR" H 5800 5200 50  0001 C CNN "MPN"
+F 4 "LMQ61460AFSQRJRRQ1" H 5800 5200 50  0001 C CNN "MPN"
 	1    5800 5200
 	1    0    0    -1
