File: Electronics/LCP_PowerControl/PowerRegulators.sch (KiCad schematic (older format))
At the start: 33 parts, among them U4 LMR50410, U5 LM61460

Commit message: LCP PowerControl Board Update
Parts:
- added D8: RB060M-60TR, Diode_SMD:D_SOD-123F, symbol Device:D_Schottky_ALT
- C17, C18, C23, C25: MPN C3225X7R1H106M250AC -> CL32B106KMVNNWE
- C19: MPN CL10A105KB8NNNC -> C1608X5R1H105K080AB
- C24: MPN C0603C105Z8VACTU -> CL10B105KP8NNNC
- C31, C32, C33: footprint Resistor_SMD:R_0603_1608Metric -> Resistor_SMD:R_0805_2012Metric; MPN C1608X5R1E106M080AC -> GRM21BR61E106KA73L
- R14: MPN CRCW040226K7FKED -> RC0402FR-0726K7L
- R17: value 22.1k -> 15k; MPN RMCF0402FT22K1 -> RC0402JR-0715KL
- R19: MPN CRCW04029K09FKED -> RT0402BRD079K09L
- U4: value LMR50410 -> BD9G102G-LB; MPN LMR50410YQDBVRQ1 -> BD9G102G-LB
Connections:
- wire segments 145 -> 148
Other:
- moved on the sheet: C26, L1, R16, R17
Changed lines of the file:
@@
 P 5200 1950
 F 0 "U4" H 5175 2315 50  0000 C CNN
-F 1 "LMR50410" H 5175 2224 50  0000 C CNN
+F 1 "BD9G102G-LB" H 5175 2224 50  0000 C CNN
 F 2 "Package_TO_SOT_SMD:SOT-23-6_Handsoldering" H 5150 1650 50  0001 C CNN
 F 3 "https://www.ti.com/lit/ds/symlink/lmr50410.pdf?ts=1591402847494&ref_url=https://www.ti.com/product/LMR50410" H 5050 2100 50  0001 C CNN
-F 4 "LMR50410YQDBVRQ1" H 5200 1950 50  0001 C CNN "MPN"
+F 4 "BD9G102G-LB" H 5200 1950 50  0001 C CNN "MPN"
 	1    5200 1950
 	1    0    0    -1
@@
 F 2 "Capacitor_SMD:C_0603_1608Metric" H 3338 1950 50  0001 C CNN
 F 3 "~" H 3300 2100 50  0001 C CNN
-F 4 "CL10A105KB8NNNC" H 3300 2100 50  0001 C CNN "MPN"
+F 4 "C1608X5R1H105K080AB" H 3300 2100 50  0001 C CNN "MPN"
 	1    3300 2100
 	1    0    0    -1
@@
 L Device:C C26
 U 1 1 5EF3B84D
-P 6350 2050
-F 0 "C26" H 6465 2096 50  0000 L CNN
-F 1 "0.1uF" H 6465 2005 50  0000 L CNN
-F 2 "Capacitor_SMD:C_0402_1005Metric" H 6465 1959 50  0001 L CNN
-F 3 "~" H 6350 2050 50  0001 C CNN
-F 4 "GRM155R71A104KA01D" H 6350 2050 50  0001 C CNN "MPN"
-	1    6350 2050
+P 6150 2050
+F 0 "C26" H 6265 2096 50  0000 L CNN
+F 1 "0.1uF" H 6265 2005 50  0000 L CNN
+F 2 "Capacitor_SMD:C_0402_1005Metric" H 6265 1959 50  0001 L CNN
+F 3 "~" H 6150 2050 50  0001 C CNN
+F 4 "GRM155R71A104KA01D" H 6150 2050 50  0001 C CNN "MPN"
+	1    6150 2050
 	1    0    0    -1
 $EndComp
@@
 $EndComp
 Wire Wire Line
-	5500 1850 6350 1850
-Wire Wire Line
-	6350 1850 6350 1900
-Wire Wire Line
-	5500 1950 6000 1950
-Wire Wire Line
-	6000 1950 6000 2250
-Wire Wire Line
-	6000 2250 6350 2250
-Wire Wire Line
-	6350 2250 6350 2200
+	5500 1850 6150 1850
+Wire Wire Line
+	6150 1850 6150 1900
+Wire Wire Line
+	5500 1950 5850 1950
+Wire Wire Line
+	5850 1950 5850 2250
+Wire Wire Line
+	5850 2250 6150 2250
+Wire Wire Line
+	6150 2250 6150 2200
 $Comp
 L Device:L L1
 U 1 1 5EF3E9E5
-P 6750 1850
-F 0 "L1" V 6940 1850 50  0000 C CNN
-F 1 "12uH" V 6849 1850 50  0000 C CNN
-F 2 "Inductor_SMD:L_Bourns-SRN8040_8x8.15mm" H 6750 1850 50  0001 C CNN
-F 3 "~" H 6750 1850 50  0001 C CNN
-F 4 "SDR0805-120ML" H 6750 1850 50  0001 C CNN "MPN"
-	1    6750 1850
+P 6950 1850
+F 0 "L1" V 7140 1850 50  0000 C CNN
+F 1 "12uH" V 7049 1850 50  0000 C CNN
+F 2 "Inductor_SMD:L_Bourns-SRN8040_8x8.15mm" H 6950 1850 50  0001 C CNN
+F 3 "~" H 6950 1850 50  0001 C CNN
+F 4 "SDR0805-120ML" H 6950 1850 50  0001 C CNN "MPN"
+	1    6950 1850
 	0    -1   -1   0
 $EndComp
 Wire Wire Line
-	6600 1850 6350 1850
-Connection ~ 6350 1850
+	6800 1850 6550 1850
+Connection ~ 6150 1850
 Wire Wire Line
 	8150 1850 8150 1900
@@
 Connection ~ 8150 1850
 Wire Wire Line
-	6900 1850 7050 1850
+	7100 1850 7250 1850
 $Comp
 L Device:R R16
 U 1 1 5EF42F65
-P 7050 2150
-F 0 "R16" H 7120 2196 50  0000 L CNN
-F 1 "51k" H 7120 2105 50  0000 L CNN
-F 2 "Resistor_SMD:R_0603_1608Metric" V 6980 2150 50  0001 C CNN
-F 3 "~" H 7050 2150 50  0001 C CNN
-F 4 "RC0603FR-0751KL" H 7050 2150 50  0001 C CNN "MPN"
-	1    7050 2150
+P 7250 2150
+F 0 "R16" H 7320 2196 50  0000 L CNN
+F 1 "51k" H 7320 2105 50  0000 L CNN
+F 2 "Resistor_SMD:R_0603_1608Metric" V 7180 2150 50  0001 C CNN
+F 3 "~" H 7250 2150 50  0001 C CNN
+F 4 "RC0603FR-0751KL" H 7250 2150 50  0001 C CNN "MPN"
+	1    7250 2150
 	1    0    0    -1
 $EndComp
@@
 L Device:R R17
 U 1 1 5EF433B6
-P 7050 2650
-F 0 "R17" H 7120 2696 50  0000 L CNN
-F 1 "22.1k" H 7120 2605 50  0000 L CNN
-F 2 "Resistor_SMD:R_0402_1005Metric" V 6980 2650 50  0001 C CNN
-F 3 "~" H 7050 2650 50  0001 C CNN
-F 4 "RMCF0402FT22K1" H 7050 2650 50  0001 C CNN "MPN"
-	1    7050 2650
+P 7250 2900
+F 0 "R17" H 7320 2946 50  0000 L CNN
+F 1 "15k" H 7320 2855 50  0000 L CNN
+F 2 "Resistor_SMD:R_0402_1005Metric" V 7180 2900 50  0001 C CNN
+F 3 "~" H 7250 2900 50  0001 C CNN
+F 4 "RC0402JR-0715KL" H 7250 2900 50  0001 C CNN "MPN"
+	1    7250 2900
 	1    0    0    -1
 $EndComp
@@
 L power:GND #PWR053
 U 1 1 5EF43697
-P 7050 2900
-F 0 "#PWR053" H 7050 2650 50  0001 C CNN
-F 1 "GND" H 7055 2727 50  0000 C CNN
-F 2 "" H 7050 2900 50  0001 C CNN
-F 3 "" H 7050 2900 50  0001 C CNN
-	1    7050 2900
-	1    0    0    -1
-$EndComp
-Wire Wire Line
-	7050 2800 7050 2900
-Wire Wire Line
-	7050 2000 7050 1850
-Connection ~ 7050 1850
-Wire Wire Line
-	7050 1850 7450 1850
+P 7250 3150
+F 0 "#PWR053" H 7250 2900 50  0001 C CNN
+F 1 "GND" H 7255 2977 50  0000 C CNN
+F 2 "" H 7250 3150 50  0001 C CNN
+F 3 "" H 7250 3150 50  0001 C CNN
+	1    7250 3150
+	1    0    0    -1
+$EndComp
+Wire Wire Line
+	7250 3050 7250 3150
+Wire Wire Line
+	7250 2000 7250 1850
+Connection ~ 7250 1850
+Wire Wire Line
+	7250 1850 7450 1850
 Wire Wire Line
 	4850 1850 4600 1850
@@
 F 2 "Capacitor_SMD:C_1210_3225Metric" H 3088 4100 50  0001 C CNN
 F 3 "~" H 3050 4250 50  0001 C CNN
-F 4 "C3225X7R1H106M250AC" H 3050 4250 50  0001 C CNN "MPN"
+F 4 "CL32B106KMVNNWE" H 3050 4250 50  0001 C CNN "MPN"
 	1    3050 4250
 	1    0    0    -1
@@
 F 2 "Capacitor_SMD:C_0603_1608Metric" H 4638 5300 50  0001 C CNN
 F 3 "~" H 4600 5450 50  0001 C CNN
-F 4 "C0603C105Z8VACTU" H 4600 5450 50  0001 C CNN "MPN"
+F 4 "CL10B105KP8NNNC" H 4600 5450 50  0001 C CNN "MPN"
 	1    4600 5450
 	1    0    0    -1
@@
 F 2 "Capacitor_SMD:C_1210_3225Metric" H 4538 4100 50  0001 C CNN
 F 3 "~" H 4500 4250 50  0001 C CNN
-F 4 "C3225X7R1H106M250AC" H 4500 4250 50  0001 C CNN "MPN"
+F 4 "CL32B106KMVNNWE" H 4500 4250 50  0001 C CNN "MPN"
 	1    4500 4250
 	1    0    0    -1
@@
 F 2 "Resistor_SMD:R_0402_1005Metric" V 4030 5450 50  0001 C CNN
 F 3 "~" H 4100 5450 50  0001 C CNN
-F 4 "CRCW040226K7FKED" H 4100 5450 50  0001 C CNN "MPN"
+F 4 "RC0402FR-0726K7L" H 4100 5450 50  0001 C CNN "MPN"
 	1    4100 5450
 	1    0    0    -1
@@
 F 2 "Resistor_SMD:R_0402_1005Metric" V 8430 5700 50  0001 C CNN
 F 3 "~" H 8500 5700 50  0001 C CNN
-F 4 "CRCW04029K09FKED" H 8500 5700 50  0001 C CNN "MPN"
+F 4 "RT0402BRD079K09L" H 8500 5700 50  0001 C CNN "MPN"
 	1    8500 5700
 	-1   0    0    1
@@
 F 0 "C31" H 9815 5346 50  0000 L CNN
 F 1 "10uF" H 9815 5255 50  0000 L CNN
-F 2 "Resistor_SMD:R_0603_1608Metric" H 9738 5150 50  0001 C CNN
+F 2 "Resistor_SMD:R_0805_2012Metric" H 9738 5150 50  0001 C CNN
 F 3 "~" H 9700 5300 50  0001 C CNN
-F 4 "C1608X5R1E106M080AC" H 9700 5300 50  0001 C CNN "MPN"
+F 4 "GRM21BR61E106KA73L" H 9700 5300 50  0001 C CNN "MPN"
 	1    9700 5300
 	1    0    0    -1
@@
 F 2 "Capacitor_SMD:C_1210_3225Metric" H 4938 4100 50  0001 C CNN
 F 3 "~" H 4900 4250 50  0001 C CNN
-F 4 "C3225X7R1H106M250AC" H 4900 4250 50  0001 C CNN "MPN"
+F 4 "CL32B106KMVNNWE" H 4900 4250 50  0001 C CNN "MPN"
 	1    4900 4250
 	1    0    0    -1
@@
 F 2 "Capacitor_SMD:C_1210_3225Metric" H 2688 4100 50  0001 C CNN
 F 3 "~" H 2650 4250 50  0001 C CNN
-F 4 "C3225X7R1H106M250AC" H 2650 4250 50  0001 C CNN "MPN"
+F 4 "CL32B106KMVNNWE" H 2650 4250 50  0001 C CNN "MPN"
 	1    2650 4250
 	1    0    0    -1
@@
 F 0 "C32" H 10215 5346 50  0000 L CNN
 F 1 "10uF" H 10215 5255 50  0000 L CNN
-F 2 "Resistor_SMD:R_0603_1608Metric" H 10138 5150 50  0001 C CNN
+F 2 "Resistor_SMD:R_0805_2012Metric" H 10138 5150 50  0001 C CNN
 F 3 "~" H 10100 5300 50  0001 C CNN
-F 4 "C1608X5R1E106M080AC" H 10100 5300 50  0001 C CNN "MPN"
+F 4 "GRM21BR61E106KA73L" H 10100 5300 50  0001 C CNN "MPN"
 	1    10100 5300
 	1    0    0    -1
@@
 F 0 "C33" H 10615 5346 50  0000 L CNN
 F 1 "10uF" H 10615 5255 50  0000 L CNN
-F 2 "Resistor_SMD:R_0603_1608Metric" H 10538 5150 50  0001 C CNN
+F 2 "Resistor_SMD:R_0805_2012Metric" H 10538 5150 50  0001 C CNN
 F 3 "~" H 10500 5300 50  0001 C CNN
-F 4 "C1608X5R1E106M080AC" H 10500 5300 50  0001 C CNN "MPN"
+F 4 "GRM21BR61E106KA73L" H 10500 5300 50  0001 C CNN "MPN"
 	1    10500 5300
 	1    0    0    -1
@@
 	10100 4950 10100 5050
 Wire Wire Line
-	7050 2300 7050 2400
-Wire Wire Line
-	7050 2400 5750 2400
-Wire Wire Line
-	5750 2400 5750 2050
+	7250 2300 7250 2650
+Wire Wire Line
+	7250 2650 5750 2650
+Wire Wire Line
+	5750 2650 5750 2050
 Wire Wire Line
 	5750 2050 5500 2050
-Connection ~ 7050 2400
-Wire Wire Line
-	7050 2400 7050 2500
+Connection ~ 7250 2650
+Wire Wire Line
+	7250 2650 7250 2750
+$Comp
+L Device:D_Schottky_ALT D8
+U 1 1 61591F94
+P 6550 2050
+F 0 "D8" V 6504 2130 50  0000 L CNN
+F 1 "RB060M-60TR" V 6650 2050 50  0000 L CNN
+F 2 "Diode_SMD:D_SOD-123F" H 6550 2050 50  0001 C CNN
+F 3 "~" H 6550 2050 50  0001 C CNN
+F 4 "RB060M-60TR" V 6550 2050 50  0001 C CNN "MPN"
+	1    6550 2050
+	0    1    1    0
+$EndComp
+Wire Wire Line
+	6550 1900 6550 1850
+Connection ~ 6550 1850
+Wire Wire Line
+	6550 1850 6150 1850
+$Comp
+L power:GND #PWR031
+U 1 1 615B7071
+P 6550 2250
+F 0 "#PWR031" H 6550 2000 50  0001 C CNN
+F 1 "GND" H 6555 2077 50  0000 C CNN
+F 2 "" H 6550 2250 50  0001 C CNN
+F 3 "" H 6550 2250 50  0001 C CNN
+	1    6550 2250
+	1    0    0    -1
+$EndComp
+Wire Wire Line
+	6550 2200 6550 2250
 $EndSCHEMATC
