File: Electronics/LCP_PowerControl/LCP_PowerControl.kicad_sch (KiCad schematic)
At the start: 0 parts

Commit message: Rev 2 Completed
Parts:
- added H1, H2, H3, H4: MountingHole_Pad, MountingHole:MountingHole_2.5mm_Pad, symbol Mechanical:MountingHole_Pad
Connections:
- new net GND: H1.1, H2.1, H3.1, H4.1
Changed lines of the file:
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@@
     (comment 2 "Updated by Joseph Kurina")
   )
+  (junction (at 52.07 184.15) (diameter 0) (color 0 0 0 0)
+  )
+  (junction (at 24.13 184.15) (diameter 0) (color 0 0 0 0)
+  )
+  (junction (at 81.28 184.15) (diameter 0) (color 0 0 0 0)
+  )
   (wire (pts (xy 55.88 97.79) (xy 109.22 97.79))
     (stroke (width 0) (type default))
   )
+  (wire (pts (xy 52.07 184.15) (xy 81.28 184.15))
+    (stroke (width 0) (type default))
+  )
+  (wire (pts (xy 24.13 184.15) (xy 24.13 187.96))
+    (stroke (width 0) (type default))
+  )
   (wire (pts (xy 238.76 107.95) (xy 243.84 107.95))
     (stroke (width 0) (type default))
@@
     (stroke (width 0) (type default))
   )
+  (wire (pts (xy 81.28 184.15) (xy 113.03 184.15))
+    (stroke (width 0) (type default))
+  )
   (wire (pts (xy 177.8 76.2) (xy 205.74 76.2))
     (stroke (width 0) (type default))
@@
     (stroke (width 0) (type default))
   )
+  (wire (pts (xy 24.13 184.15) (xy 52.07 184.15))
+    (stroke (width 0) (type default))
+  )
   (wire (pts (xy 109.22 151.13) (xy 55.88 151.13))
     (stroke (width 0) (type default))
@@
     (stroke (width 0) (type default))
   )
+  (symbol (lib_id "Mechanical:MountingHole_Pad") (at 52.07 181.61 0) (unit 1)
+    (in_bom yes) (on_board yes) (dnp no) (fields_autoplaced)
+    (property "Reference" "H2" (at 54.61 179.07 0)
+      (effects (font (size 1.27 1.27)) (justify left))
+    )
+    (property "Value" "MountingHole_Pad" (at 54.61 181.61 0)
+      (effects (font (size 1.27 1.27)) (justify left))
+    )
+    (property "Footprint" "MountingHole:MountingHole_2.5mm_Pad" (at 52.07 181.61 0)
+      (effects (font (size 1.27 1.27)) hide)
+    )
+    (property "Datasheet" "~" (at 52.07 181.61 0)
+      (effects (font (size 1.27 1.27)) hide)
+    )
+    (pin "1")
+    (instances
+      (project "LCP_PowerControl"
+        (path "/41d9a78b-a4de-4258-a1a2-a19eb582c73a"
+          (reference "H2") (unit 1)
+        )
+      )
+    )
+  )
+  (symbol (lib_id "Mechanical:MountingHole_Pad") (at 81.28 181.61 0) (unit 1)
+    (in_bom yes) (on_board yes) (dnp no) (fields_autoplaced)
+    (property "Reference" "H3" (at 83.82 179.07 0)
+      (effects (font (size 1.27 1.27)) (justify left))
+    )
+    (property "Value" "MountingHole_Pad" (at 83.82 181.61 0)
+      (effects (font (size 1.27 1.27)) (justify left))
+    )
+    (property "Footprint" "MountingHole:MountingHole_2.5mm_Pad" (at 81.28 181.61 0)
+      (effects (font (size 1.27 1.27)) hide)
+    )
+    (property "Datasheet" "~" (at 81.28 181.61 0)
+      (effects (font (size 1.27 1.27)) hide)
+    )
+    (pin "1")
+    (instances
+      (project "LCP_PowerControl"
+        (path "/41d9a78b-a4de-4258-a1a2-a19eb582c73a"
+          (reference "H3") (unit 1)
+        )
+      )
+    )
+  )
+  (symbol (lib_id "Mechanical:MountingHole_Pad") (at 24.13 181.61 0) (unit 1)
+    (in_bom yes) (on_board yes) (dnp no) (fields_autoplaced)
+    (property "Reference" "H1" (at 26.67 179.07 0)
+      (effects (font (size 1.27 1.27)) (justify left))
+    )
+    (property "Value" "MountingHole_Pad" (at 26.67 181.61 0)
+      (effects (font (size 1.27 1.27)) (justify left))
+    )
+    (property "Footprint" "MountingHole:MountingHole_2.5mm_Pad" (at 24.13 181.61 0)
+      (effects (font (size 1.27 1.27)) hide)
+    )
+    (property "Datasheet" "~" (at 24.13 181.61 0)
+      (effects (font (size 1.27 1.27)) hide)
+    )
+    (pin "1")
+    (instances
+      (project "LCP_PowerControl"
+        (path "/41d9a78b-a4de-4258-a1a2-a19eb582c73a"
+          (reference "H1") (unit 1)
+        )
+      )
+    )
+  )
+  (symbol (lib_id "power:GND") (at 24.13 187.96 0) (unit 1)
+    (in_bom yes) (on_board yes) (dnp no) (fields_autoplaced)
+    (property "Reference" "#PWR033" (at 24.13 194.31 0)
+      (effects (font (size 1.27 1.27)) hide)
+    )
+    (property "Value" "GND" (at 24.13 193.04 0)
+      (effects (font (size 1.27 1.27)))
+    )
+    (property "Footprint" "" (at 24.13 187.96 0)
+      (effects (font (size 1.27 1.27)) hide)
+    )
+    (property "Datasheet" "" (at 24.13 187.96 0)
+      (effects (font (size 1.27 1.27)) hide)
+    )
+    (pin "1")
+    (instances
+      (project "LCP_PowerControl"
+        (path "/41d9a78b-a4de-4258-a1a2-a19eb582c73a"
+          (reference "#PWR033") (unit 1)
+        )
+      )
+    )
+  )
+  (symbol (lib_id "Mechanical:MountingHole_Pad") (at 113.03 181.61 0) (unit 1)
+    (in_bom yes) (on_board yes) (dnp no) (fields_autoplaced)
+    (property "Reference" "H4" (at 115.57 179.07 0)
+      (effects (font (size 1.27 1.27)) (justify left))
+    )
+    (property "Value" "MountingHole_Pad" (at 115.57 181.61 0)
+      (effects (font (size 1.27 1.27)) (justify left))
+    )
+    (property "Footprint" "MountingHole:MountingHole_2.5mm_Pad" (at 113.03 181.61 0)
+      (effects (font (size 1.27 1.27)) hide)
+    )
+    (property "Datasheet" "~" (at 113.03 181.61 0)
+      (effects (font (size 1.27 1.27)) hide)
+    )
+    (pin "1")
+    (instances
+      (project "LCP_PowerControl"
+        (path "/41d9a78b-a4de-4258-a1a2-a19eb582c73a"
+          (reference "H4") (unit 1)
+        )
+      )
+    )
+  )
   (sheet (at 21.59 21.59) (size 34.29 29.21) (fields_autoplaced)
